File: eagle/Filter/Filter/Filter.brd (EAGLE design)
At the start: 50.5 x 48.2 mm, 13 parts, among them IC1 TDA2320AP, X1 R_PASS, X2 C_PASS, X6 ACT_OUT, X7 PASS_OUT

Commit message: Fixed filter files, fixed molex on eagle board
Parts:
- ACT_IN, PASS_IN, VCC_5V, V_REF: value (none) -> 22-23-2021; device con-molex:KK-156-2 -> con-molex:22-23-2021
- X6, X7: device con-molex:KK-156-2 -> con-molex:22-23-2021
Routing:
- net V_REF: track 25.1 -> 25.8 mm
- net VCC: track 29.3 -> 30.0 mm
- net PASS_OUT: track 23.9 -> 23.2 mm
- net ACT_OUT: track 38.6 -> 39.3 mm
- net ACT_IN: track 20.0 -> 20.7 mm
- net PASS_IN: track 15.8 -> 15.1 mm
Changed lines of the file:
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@@
 </element>
 <element name="IC1" library="linear" package="DIL08" value="TDA2320AP" x="27.94" y="25.4" rot="R180"/>
-<element name="ACT_IN" library="con-molex" package="KK-156-2" value="" x="7.62" y="41.91" rot="R270">
-<attribute name="OC_NEWARK" value="unknown" x="2.54" y="24.13" size="1.778" layer="27" rot="R270" display="off"/>
-<attribute name="MPN" value="" x="2.54" y="24.13" size="1.778" layer="27" rot="R270" display="off"/>
-<attribute name="MF" value="" x="2.54" y="24.13" size="1.778" layer="27" rot="R270" display="off"/>
-<attribute name="OC_FARNELL" value="unknown" x="2.54" y="24.13" size="1.778" layer="27" rot="R270" display="off"/>
+<element name="ACT_IN" library="con-molex" package="22-23-2021" value="22-23-2021" x="7.62" y="41.91" rot="R270">
+<attribute name="OC_NEWARK" value="25C3832" x="2.54" y="24.13" size="1.778" layer="27" rot="R270" display="off"/>
+<attribute name="MPN" value="22-23-2021" x="2.54" y="24.13" size="1.778" layer="27" rot="R270" display="off"/>
+<attribute name="MF" value="MOLEX" x="2.54" y="24.13" size="1.778" layer="27" rot="R270" display="off"/>
+<attribute name="OC_FARNELL" value="1462926" x="2.54" y="24.13" size="1.778" layer="27" rot="R270" display="off"/>
 </element>
-<element name="VCC_5V" library="con-molex" package="KK-156-2" value="" x="7.62" y="19.05" rot="R270">
-<attribute name="OC_NEWARK" value="unknown" x="2.54" y="-19.05" size="1.778" layer="27" rot="R270" display="off"/>
-<attribute name="MPN" value="" x="2.54" y="-19.05" size="1.778" layer="27" rot="R270" display="off"/>
-<attribute name="MF" value="" x="2.54" y="-19.05" size="1.778" layer="27" rot="R270" display="off"/>
-<attribute name="OC_FARNELL" value="unknown" x="2.54" y="-19.05" size="1.778" layer="27" rot="R270" display="off"/>
+<element name="VCC_5V" library="con-molex" package="22-23-2021" value="22-23-2021" x="7.62" y="19.05" rot="R270">
+<attribute name="OC_NEWARK" value="25C3832" x="2.54" y="-19.05" size="1.778" layer="27" rot="R270" display="off"/>
+<attribute name="MPN" value="22-23-2021" x="2.54" y="-19.05" size="1.778" layer="27" rot="R270" display="off"/>
+<attribute name="MF" value="MOLEX" x="2.54" y="-19.05" size="1.778" layer="27" rot="R270" display="off"/>
+<attribute name="OC_FARNELL" value="1462926" x="2.54" y="-19.05" size="1.778" layer="27" rot="R270" display="off"/>
 </element>
-<element name="PASS_IN" library="con-molex" package="KK-156-2" value="" x="7.62" y="7.62" rot="R270">
-<attribute name="OC_NEWARK" value="unknown" x="2.54" y="-20.32" size="1.778" layer="27" rot="R270" display="off"/>
-<attribute name="MPN" value="" x="2.54" y="-20.32" size="1.778" layer="27" rot="R270" display="off"/>
-<attribute name="MF" value="" x="2.54" y="-20.32" size="1.778" layer="27" rot="R270" display="off"/>
-<attribute name="OC_FARNELL" value="unknown" x="2.54" y="-20.32" size="1.778" layer="27" rot="R270" display="off"/>
+<element name="PASS_IN" library="con-molex" package="22-23-2021" value="22-23-2021" x="7.62" y="7.62" rot="R270">
+<attribute name="OC_NEWARK" value="25C3832" x="2.54" y="-20.32" size="1.778" layer="27" rot="R270" display="off"/>
+<attribute name="MPN" value="22-23-2021" x="2.54" y="-20.32" size="1.778" layer="27" rot="R270" display="off"/>
+<attribute name="MF" value="MOLEX" x="2.54" y="-20.32" size="1.778" layer="27" rot="R270" display="off"/>
+<attribute name="OC_FARNELL" value="1462926" x="2.54" y="-20.32" size="1.778" layer="27" rot="R270" display="off"/>
 </element>
-<element name="X6" library="con-molex" package="KK-156-2" value="ACT_OUT" x="41.91" y="41.91" rot="R90">
-<attribute name="OC_NEWARK" value="unknown" x="57.15" y="59.69" size="1.778" layer="27" rot="R90" display="off"/>
-<attribute name="MPN" value="" x="57.15" y="59.69" size="1.778" layer="27" rot="R90" display="off"/>
-<attribute name="MF" value="" x="57.15" y="59.69" size="1.778" layer="27" rot="R90" display="off"/>
-<attribute name="OC_FARNELL" value="unknown" x="57.15" y="59.69" size="1.778" layer="27" rot="R90" display="off"/>
+<element name="X6" library="con-molex" package="22-23-2021" value="ACT_OUT" x="41.91" y="41.91" rot="R90">
+<attribute name="OC_NEWARK" value="25C3832" x="57.15" y="59.69" size="1.778" layer="27" rot="R90" display="off"/>
+<attribute name="MPN" value="22-23-2021" x="57.15" y="59.69" size="1.778" layer="27" rot="R90" display="off"/>
+<attribute name="MF" value="MOLEX" x="57.15" y="59.69" size="1.778" layer="27" rot="R90" display="off"/>
+<attribute name="OC_FARNELL" value="1462926" x="57.15" y="59.69" size="1.778" layer="27" rot="R90" display="off"/>
 </element>
-<element name="X7" library="con-molex" package="KK-156-2" value="PASS_OUT" x="41.91" y="7.62" rot="R90">
-<attribute name="OC_NEWARK" value="unknown" x="57.15" y="35.56" size="1.778" layer="27" rot="R90" display="off"/>
-<attribute name="MPN" value="" x="57.15" y="35.56" size="1.778" layer="27" rot="R90" display="off"/>
-<attribute name="MF" value="" x="57.15" y="35.56" size="1.778" layer="27" rot="R90" display="off"/>
-<attribute name="OC_FARNELL" value="unknown" x="57.15" y="35.56" size="1.778" layer="27" rot="R90" display="off"/>
+<element name="X7" library="con-molex" package="22-23-2021" value="PASS_OUT" x="41.91" y="7.62" rot="R90">
+<attribute name="OC_NEWARK" value="25C3832" x="57.15" y="35.56" size="1.778" layer="27" rot="R90" display="off"/>
+<attribute name="MPN" value="22-23-2021" x="57.15" y="35.56" size="1.778" layer="27" rot="R90" display="off"/>
+<attribute name="MF" value="MOLEX" x="57.15" y="35.56" size="1.778" layer="27" rot="R90" display="off"/>
+<attribute name="OC_FARNELL" value="1462926" x="57.15" y="35.56" size="1.778" layer="27" rot="R90" display="off"/>
 </element>
 <element name="C1" library="capacitor-wima" package="C5B3" value="100nF" x="15.24" y="19.05" rot="R90"/>
-<element name="V_REF" library="con-molex" package="KK-156-2" value="" x="7.62" y="30.48" rot="R270">
-<attribute name="OC_NEWARK" value="unknown" x="7.62" y="30.48" size="1.9304" layer="27" rot="R270" display="off"/>
-<attribute name="MPN" value="" x="7.62" y="30.48" size="1.9304" layer="27" rot="R270" display="off"/>
-<attribute name="MF" value="" x="7.62" y="30.48" size="1.9304" layer="27" rot="R270" display="off"/>
-<attribute name="OC_FARNELL" value="unknown" x="7.62" y="30.48" size="1.9304" layer="27" rot="R270" display="off"/>
+<element name="V_REF" library="con-molex" package="22-23-2021" value="22-23-2021" x="7.62" y="30.48" rot="R270">
+<attribute name="OC_NEWARK" value="25C3832" x="7.62" y="30.48" size="1.9304" layer="27" rot="R270" display="off"/>
+<attribute name="MPN" value="22-23-2021" x="7.62" y="30.48" size="1.9304" layer="27" rot="R270" display="off"/>
+<attribute name="MF" value="MOLEX" x="7.62" y="30.48" size="1.9304" layer="27" rot="R270" display="off"/>
+<attribute name="OC_FARNELL" value="1462926" x="7.62" y="30.48" size="1.9304" layer="27" rot="R270" display="off"/>
 </element>
 <element name="C2" library="capacitor-wima" package="C5B3" value="100nF" x="15.24" y="30.48" rot="R90"/>
@@
 <wire x1="15.24" y1="21.59" x2="19.05" y2="17.78" width="1.524" layer="16"/>
 <wire x1="15.24" y1="21.59" x2="7.62" y2="21.59" width="1.524" layer="16"/>
-<wire x1="7.62" y1="21.59" x2="7.62" y2="21.03" width="1.524" layer="16"/>
+<wire x1="7.62" y1="21.59" x2="7.62" y2="20.32" width="1.524" layer="16"/>
 </signal>
 <signal name="N$2">
@@
 <wire x1="10.16" y1="44.45" x2="20.32" y2="34.29" width="1.524" layer="16"/>
 <wire x1="7.62" y1="44.45" x2="10.16" y2="44.45" width="1.524" layer="16"/>
-<wire x1="7.62" y1="44.45" x2="7.62" y2="43.89" width="1.524" layer="16"/>
+<wire x1="7.62" y1="44.45" x2="7.62" y2="43.18" width="1.524" layer="16"/>
 </signal>
 <signal name="GND">
@@
 <wire x1="7.62" y1="8.89" x2="10.16" y2="11.43" width="1.524" layer="16"/>
 <wire x1="20.32" y1="8.89" x2="20.32" y2="8.62" width="1.524" layer="16"/>
-<wire x1="7.62" y1="8.89" x2="7.62" y2="9.6" width="1.524" layer="16"/>
 </signal>
 <signal name="ACT_OUT">
@@
 <wire x1="41.91" y1="39.37" x2="36.83" y2="34.29" width="1.524" layer="16"/>
 <wire x1="36.83" y1="34.29" x2="31.75" y2="29.21" width="1.524" layer="16"/>
-<wire x1="41.91" y1="39.37" x2="41.91" y2="39.93" width="1.524" layer="16"/>
+<wire x1="41.91" y1="39.37" x2="41.91" y2="40.64" width="1.524" layer="16"/>
 <wire x1="25.4" y1="41.91" x2="22.86" y2="39.37" width="1.524" layer="16"/>
 <wire x1="34.29" y1="41.91" x2="25.4" y2="41.91" width="1.524" layer="16"/>
@@
 <wire x1="15.24" y1="33.02" x2="22.86" y2="25.4" width="1.524" layer="16"/>
 <wire x1="15.24" y1="33.02" x2="7.62" y2="33.02" width="1.524" layer="16"/>
-<wire x1="7.62" y1="33.02" x2="7.62" y2="32.46" width="1.524" layer="16"/>
+<wire x1="7.62" y1="33.02" x2="7.62" y2="31.75" width="1.524" layer="16"/>
 </signal>
 <signal name="PASS_OUT">
@@
 <wire x1="20.32" y1="6.35" x2="20.32" y2="6.62" width="1.524" layer="16"/>
 <wire x1="29.21" y1="6.35" x2="41.91" y2="6.35" width="1.524" layer="16"/>
-<wire x1="41.91" y1="6.35" x2="41.91" y2="5.64" width="1.524" layer="16"/>
 <wire x1="29.21" y1="6.35" x2="29.21" y2="6.62" width="1.524" layer="16"/>
 </signal>
