File: eagle/Filter/Filter/Filter.sch (EAGLE design)
At the start: 13 parts, among them IC1 TDA2320AP, X1 R_PASS, X2 C_PASS, X6 ACT_OUT, X7 PASS_OUT

Commit message: Fixed filter files, fixed molex on eagle board
Parts:
- ACT_IN, PASS_IN, VCC_5V, V_REF: value (none) -> 22-23-2021; device con-molex:KK-156-2 -> con-molex:22-23-2021
- X6, X7: device con-molex:KK-156-2 -> con-molex:22-23-2021
Changed lines of the file:
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@@
 <part name="GND1" library="supply1" deviceset="GND" device=""/>
 <part name="P+1" library="supply1" deviceset="VCC" device=""/>
-<part name="ACT_IN" library="con-molex" deviceset="KK-156-2" device=""/>
-<part name="VCC_5V" library="con-molex" deviceset="KK-156-2" device=""/>
-<part name="PASS_IN" library="con-molex" deviceset="KK-156-2" device=""/>
-<part name="X6" library="con-molex" deviceset="KK-156-2" device="" value="ACT_OUT"/>
-<part name="X7" library="con-molex" deviceset="KK-156-2" device="" value="PASS_OUT"/>
+<part name="ACT_IN" library="con-molex" deviceset="22-23-2021" device=""/>
+<part name="VCC_5V" library="con-molex" deviceset="22-23-2021" device=""/>
+<part name="PASS_IN" library="con-molex" deviceset="22-23-2021" device=""/>
+<part name="X6" library="con-molex" deviceset="22-23-2021" device="" value="ACT_OUT"/>
+<part name="X7" library="con-molex" deviceset="22-23-2021" device="" value="PASS_OUT"/>
 <part name="GND2" library="supply1" deviceset="GND" device=""/>
 <part name="GND3" library="supply1" deviceset="GND" device=""/>
@@
 <part name="C1" library="capacitor-wima" deviceset="C" device="5/3" value="100nF"/>
 <part name="GND9" library="supply1" deviceset="GND" device=""/>
-<part name="V_REF" library="con-molex" deviceset="KK-156-2" device=""/>
+<part name="V_REF" library="con-molex" deviceset="22-23-2021" device=""/>
 <part name="C2" library="capacitor-wima" deviceset="C" device="5/3" value="100nF"/>
 <part name="GND5" library="supply1" deviceset="GND" device=""/>
